File: ROV Control 1.brd (EAGLE design)
At the start: 160 x 100 mm, 6 parts, among them J4 RASPBERRYPI-40-PIN-GPIO_PTH, U1 ARDUINOR3-BPLACE, X1 S4B-ZR

Commit message: Add files via upload
Parts:
- added R1, R2, R3: 10k, SparkFun-Resistors:0603
- added R4, R5, R6: 1k, SparkFun-Resistors:0603
- moved J3 4.58 mm to (74.9, 66.0)
- moved J2 3.59 mm to (86.4, 66.0), turned to 180 degrees
- moved J1 2.54 mm to (92.7, 66.0)
Connections:
- new net 12V: R1.1, R2.1, R3.1
- new net N$10: R3.2, R6.2, U1.D7
- new net N$9: R2.2, R5.2, U1.D6
- net GND: now also R4.1, R5.1, R6.1
- net N$7: now also R1.2, R4.2, U1.D5; no longer X1.1
Routing:
- net GND: track 0.00 -> 116.3 mm
- net 5V: track 0.00 -> 31.6 mm
- net N$9: track 0.00 -> 25.0 mm
- net 3.3V: track 0.00 -> 21.3 mm
- net N$7: track 0.00 -> 18.4 mm
- net N$10: track 0.00 -> 17.6 mm
- net N$3: track 0.00 -> 15.4 mm
- net N$4: track 0.00 -> 15.2 mm
- net N$2: track 0.00 -> 13.9 mm
- net 12V: track 0.00 -> 8.98 mm
- net N$6: track 0.00 -> 7.15 mm
- net N$5: track 0.00 -> 6.67 mm
- net N$1: track 0.00 -> 6.52 mm
Other:
- outline, holes or cut-outs redrawn

Commit message: Add files via upload
Parts:
- removed J1, J2, J3: (no value), SparkFun-Connectors:1X03
- added J5, J6, J7: (no value), SparkFun-Connectors:1X03
Connections:
- net GND: now also J5.3, J6.3, J7.3; no longer J1.3, J2.3, J3.3
- net N$2: now also J6.1; no longer J2.1
- net N$3: now also J5.1; no longer J1.1
- net N$4: now also J7.1; no longer J3.1
Routing:
- net GND: track 116.3 -> 0.00 mm
- net 5V: track 31.6 -> 0.00 mm
- net N$9: track 25.0 -> 0.00 mm
- net 3.3V: track 21.3 -> 0.00 mm
- net N$7: track 18.4 -> 0.00 mm
- net N$10: track 17.6 -> 0.00 mm
- net N$3: track 15.4 -> 0.00 mm
- net N$4: track 15.2 -> 0.00 mm
- net N$2: track 13.9 -> 0.00 mm
- net 12V: track 8.98 -> 0.00 mm
- net N$6: track 7.15 -> 0.00 mm
- net N$5: track 6.67 -> 0.00 mm
- net N$1: track 6.52 -> 0.00 mm
