File: ROV Control 1.sch (EAGLE design)
At the start: 6 parts, among them J4 RASPBERRYPI-40-PIN-GPIO_PTH, U1 ARDUINOR3-BPLACE, X1 S4B-ZR

Commit message: Add files via upload
Parts:
- added R1, R2, R3: 10k, SparkFun-Resistors:10KOHM-0603-1/10W-1%
- added R4, R5, R6: 1k, SparkFun-Resistors:1KOHM-0603-1/10W-1%
Connections:
- new net 12V: R1.1, R2.1, R3.1
- new net N$10: R3.2, R6.2, U1.D7
- new net N$9: R2.2, R5.2, U1.D6
- net GND: now also R4.1, R5.1, R6.1
- net N$7: now also R1.2, R4.2, U1.D5; no longer X1-1.1
Other:
- moved on the sheet: J4

Commit message: Add files via upload
Parts:
- removed J1: (no value), SparkFun-Connectors:CONN_03
- added J5, J6, J7: (no value), SparkFun-Connectors:CONN_03
Connections:
- net GND: no longer J1.3
- net N$3: no longer J1.1
Changed lines of the file:
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@@
 <parts>
 <part name="U1" library="adafruit" library_urn="urn:adsk.eagle:library:420" deviceset="ARDUINOR3" device="-BPLACE"/>
-<part name="J1" library="SparkFun-Connectors" library_urn="urn:adsk.eagle:library:513" deviceset="CONN_03" device="" package3d_urn="urn:adsk.eagle:package:38063/1"/>
 <part name="GND2" library="SparkFun-PowerSymbols" library_urn="urn:adsk.eagle:library:530" deviceset="GND" device=""/>
 <part name="J2" library="SparkFun-Connectors" library_urn="urn:adsk.eagle:library:513" deviceset="CONN_03" device="" package3d_urn="urn:adsk.eagle:package:38063/1"/>
@@
 <part name="SUPPLY2" library="SparkFun-PowerSymbols" library_urn="urn:adsk.eagle:library:530" deviceset="12V" device=""/>
 <part name="SUPPLY3" library="SparkFun-PowerSymbols" library_urn="urn:adsk.eagle:library:530" deviceset="12V" device=""/>
+<part name="J5" library="SparkFun-Connectors" library_urn="urn:adsk.eagle:library:513" deviceset="CONN_03" device="" package3d_urn="urn:adsk.eagle:package:38063/1"/>
+<part name="J6" library="SparkFun-Connectors" library_urn="urn:adsk.eagle:library:513" deviceset="CONN_03" device="" package3d_urn="urn:adsk.eagle:package:38063/1"/>
+<part name="J7" library="SparkFun-Connectors" library_urn="urn:adsk.eagle:library:513" deviceset="CONN_03" device="" package3d_urn="urn:adsk.eagle:package:38063/1"/>
 </parts>
 <sheets>
@@
 <instances>
 <instance part="U1" gate="G$1" x="99.06" y="12.7"/>
-<instance part="J1" gate="J$1" x="139.7" y="45.72" rot="R90"/>
 <instance part="GND2" gate="1" x="137.16" y="58.42" rot="R180"/>
 <instance part="J2" gate="J$1" x="160.02" y="45.72" rot="R90"/>
@@
 <instance part="SUPPLY2" gate="G$1" x="182.88" y="-33.02" rot="R180"/>
 <instance part="SUPPLY3" gate="G$1" x="205.74" y="-33.02" rot="R180"/>
+<instance part="J5" gate="J$1" x="160.02" y="27.94" rot="R90"/>
+<instance part="J6" gate="J$1" x="177.8" y="27.94" rot="R90"/>
+<instance part="J7" gate="J$1" x="200.66" y="27.94" rot="R90"/>
 </instances>
 <busses>
@@
 <net name="GND" class="0">
 <segment>
-<pinref part="J1" gate="J$1" pin="3"/>
 <pinref part="GND2" gate="1" pin="GND"/>
 <wire x1="137.16" y1="55.88" x2="137.16" y2="53.34" width="0.1524" layer="91"/>
@@
 <wire x1="132.08" y1="53.34" x2="132.08" y2="43.18" width="0.1524" layer="91"/>
 <wire x1="132.08" y1="43.18" x2="134.62" y2="40.64" width="0.1524" layer="91"/>
-<pinref part="J1" gate="J$1" pin="1"/>
 <wire x1="142.24" y1="53.34" x2="147.32" y2="53.34" width="0.1524" layer="91"/>
 <wire x1="147.32" y1="53.34" x2="147.32" y2="40.64" width="0.1524" layer="91"/>
