File: Control board V4.brd (EAGLE design)
At the start: 68.6 x 53.3 mm, 12 parts, among them CN1 1X4-BIG, J1 RASPBERRYPI-40-PIN-GPIO_PTH_N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

Commit message: Add files via upload
Parts:
- moved R5 12.7 mm to (71.1, 29.2)
- moved J6 10.9 mm to (68.6, 48.3)
- moved J5 10.2 mm to (95.2, 48.3)
- moved R6 7.62 mm to (81.3, 29.2)
- moved R9 7.62 mm to (76.2, 17.8)
- moved J7 6.84 mm to (85.1, 48.3)
- moved R7 3.81 mm to (97.8, 17.8)
- moved R4 2.54 mm to (91.4, 29.2)
- moved R8 2.54 mm to (86.4, 17.8)
Connections:
- new net N$1: J1.5, U$1.A4
- new net N$9: J1.3, U$1.A5
Routing:
- net GND: track 185.0 -> 0.00 mm
- net 5V: track 43.0 -> 0.00 mm
- net N$6: track 31.1 -> 0.00 mm
- net N$11: track 30.7 -> 0.00 mm
- net N$5: track 26.7 -> 0.00 mm
- net N$7: track 25.8 -> 0.00 mm
- net N$4: track 24.2 -> 0.00 mm
- net N$10: track 18.6 -> 0.00 mm
- net N$2: track 14.2 -> 0.00 mm
- net N$8: track 9.14 -> 0.00 mm
- net N$3: track 6.77 -> 0.00 mm
