File: Control board V5.brd (EAGLE design)
At the start: 68.6 x 53.3 mm, 12 parts, among them CN1 1X4-BIG, J1 RASPBERRYPI-40-PIN-GPIO_PTH_N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

Commit message: Add files via upload
Parts:
- moved J5 5.08 mm to (90.2, 49.5), turned to 180 degrees
- moved R4 1.27 mm to (94.0, 27.9)
- moved R5 1.27 mm to (83.8, 27.9)
- moved R6 1.27 mm to (88.9, 27.9)
Connections:
- new net N$1: J1.5, U$1.A4
- new net N$9: J1.3, U$1.A5
Routing:
- net N$9: track 0.00 -> 61.2 mm, vias 0 -> 1
- net N$1: track 0.00 -> 56.9 mm, vias 0 -> 1
- net GND: track 185.0 -> 168.7 mm
- net N$7: track 25.8 -> 32.0 mm
- net N$8: track 9.14 -> 11.1 mm
- net N$6: track 31.1 -> 29.3 mm
- net 5V: track 43.0 -> 44.7 mm, vias 0 -> 1
- net N$10: track 18.6 -> 16.9 mm
- net N$4: track 24.2 -> 23.2 mm
- net N$5: track 26.7 -> 25.7 mm
- net N$11: track 30.7 -> 29.8 mm
